File: topo/ATTiny Fuse Reset with 12V Charge Pump.brd (EAGLE design)
At the start: 68.6 x 53.3 mm, 57 parts, among them SW4 SWITCH_SPDT, U1 ARDUINOR3-BPLACE

Commit message: adde pdf
Routing:
- net N$2: track 31.0 -> 31.8 mm
- net GND: track 233.7 -> 234.5 mm
